File: hardware/GPS.kicad_sch (KiCad schematic)
At the start: 8 parts, among them U2 MAX-M10S

Commit message: Added PPG schematic page
Parts:
- added TP10, TP3, TP4, TP5, TP6, TP7, TP8, TP9: TestPoint, symbol Connector:TestPoint
- C16, C17: value 100nF -> C
Connections:
- net +3V3: now also TP10.1
- net MAX_M10_LNA_EN: now also TP8.1
- net MAX_M10_SCL: now also TP7.1
- net MAX_M10_SDA: now also TP6.1
- net MAX_M10_VIO_SEL_NC: now also TP5.1
- net MAX_M10_nRST: now also TP9.1
- net MAX_M10_SAFEBOOT: now reaches U2.18 (~{SAFEBOOT})
- net MAX_M10_SAFEBOOT: now also TP3.1
- net MAX_M10_TIMEPULSE: now reaches U2.4 (TIMEPULSE)
- net MAX_M10_TIMEPULSE: now also TP4.1
- net MAX_M10_HOST_CTL: now reaches U2.5 (EXTINT)
- no-connect marks 4 -> 3
Other:
- note added: "For 3p3 leave VIO_SEL NC"
- note added: "I2C must run at 400kHz"
- note removed: "TODO: Do I need a SAW filter?"
- moved on the sheet: AE1, C16, C17, L2

Commit message: Added bluetooth module schematic and environmental perception block"
Other:
- note added: "TODO: Should I put a load switch in between the power supply and this device? - Footprint of a lsw is very small, and would require 1 GPIO from STM to actuate Software standby mode is 46uA, which is pretty large How is GPS data turned into a GPX file?"
Changed lines of the file:
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@@
+		)
+	)
+	(text "TODO:\nShould I put a load switch in between the power supply and this device?\n- Footprint of a lsw is very small, and would require 1 GPIO from STM to actuate\nSoftware standby mode is 46uA, which is pretty large\nHow is GPS data turned into a GPX file?"
+		(exclude_from_sim no)
+		(at 178.308 171.958 0)
+		(effects
+			(font
+				(size 1.27 1.27)
+			)
+			(justify left)
 		)
 	)

Commit message: Changing barometer, STM32 and power rails
Other:
- note added: "TODO: Should I put a load switch in between the power supply and this device? - Footprint of a lsw is very small, and would require 1 GPIO from STM to actuate Software standby mode is 46uA, which is pretty large How is GPS data turned into a GPX file? Compatible with 1p8V"
- note removed: "TODO: Should I put a load switch in between the power supply and this device? - Footprint of a lsw is very small, and would require 1 GPIO from STM to actuate Software standby mode is 46uA, which is pretty large How is GPS data turned into a GPX file?"
Changed lines of the file:
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@@
 		)
 	)
-	(text "TODO:\nShould I put a load switch in between the power supply and this device?\n- Footprint of a lsw is very small, and would require 1 GPIO from STM to actuate\nSoftware standby mode is 46uA, which is pretty large\nHow is GPS data turned into a GPX file?"
+	(text "TODO:\nShould I put a load switch in between the power supply and this device?\n- Footprint of a lsw is very small, and would require 1 GPIO from STM to actuate\nSoftware standby mode is 46uA, which is pretty large\nHow is GPS data turned into a GPX file?\nCompatible with 1p8V"
 		(exclude_from_sim no)
-		(at 178.308 171.958 0)
+		(at 178.308 173.736 0)
 		(effects
 			(font

Commit message: Added optical front end submodule and reconnected to STM32
Parts:
- removed TP5: TestPoint, symbol Connector:TestPoint
Connections:
- net MAX_M10_VIO_SEL_NC is gone; now on net GND: U2.15 (VIO_SEL)
- net +3V3 renamed +1V8
Other:
- note added: "For 1p8 GND VIO_SEL"
- note removed: "For 3p3 leave VIO_SEL NC"
