File: hardware/eMMC.kicad_sch (KiCad schematic)
At the start: 13 parts, among them IC1 MX52LM04A11XSI

Commit message: Updated schematic to add STM32
Parts:
- added unit 2 of IC1
- added unit 1 of IC1
Connections:
- net CLK: now also IC1.M6 (CLK); no longer IC1.M6 (CLK)
- net CMD: now also IC1.M5 (CMD); no longer IC1.M5 (CMD)
- net DAT0: now also IC1.A3 (DAT0); no longer IC1.A3 (DAT0)
- net DAT1: now also IC1.A4 (DAT1); no longer IC1.A4 (DAT1)
- net DAT2: now also IC1.A5 (DAT2); no longer IC1.A5 (DAT2)
- net DAT3: now also IC1.B2 (DAT3); no longer IC1.B2 (DAT3)
- net DAT4: now also IC1.B3 (DAT4); no longer IC1.B3 (DAT4)
- net DAT5: now also IC1.B4 (DAT5); no longer IC1.B4 (DAT5)
- net DAT6: now also IC1.B5 (DAT6); no longer IC1.B5 (DAT6)
- net DAT7: now also IC1.B6 (DAT7); no longer IC1.B6 (DAT7)
- net DATA_STROBE: now also IC1.H5 (DATA_STROBE); no longer IC1.H5 (DATA_STROBE)
- net GND: now also IC1.A6 (VSS_1), IC1.C4 (VSSQ_1), IC1.E7 (VSS_2), IC1.G5 (VSS_3), IC1.H10 (VSS_4), IC1.J5 (VSS_5), IC1.K8 (VSS_6), IC1.N2 (VSSQ_2), IC1.N5 (VSSQ_3), IC1.P4 (VSSQ_4), IC1.P6 (VSSQ_5); no longer IC1.A6 (VSS_1), IC1.C4 (VSSQ_1), IC1.E7 (VSS_2), IC1.G5 (VSS_3), IC1.H10 (VSS_4), IC1.J5 (VSS_5), IC1.K8 (VSS_6), IC1.N2 (VSSQ_2), IC1.N5 (VSSQ_3), IC1.P4 (VSSQ_4), IC1.P6 (VSSQ_5)
- net RFU_10_NC: now also IC1.K7 (RFU_10); no longer IC1.K7 (RFU_10)
- net RFU_11_NC: now also IC1.K10 (RFU_11); no longer IC1.K10 (RFU_11)
- net RFU_12_NC: now also IC1.P7 (RFU_12); no longer IC1.P7 (RFU_12)
- net RFU_13_NC: now also IC1.P10 (RFU_13); no longer IC1.P10 (RFU_13)
- net RFU_1_NC: now also IC1.A7 (RFU_1); no longer IC1.A7 (RFU_1)
- net RFU_2_NC: now also IC1.E5 (RFU_2); no longer IC1.E5 (RFU_2)
- net RFU_3_NC: now also IC1.E8 (RFU_3); no longer IC1.E8 (RFU_3)
- net RFU_4_NC: now also IC1.E9 (RFU_4); no longer IC1.E9 (RFU_4)
- net RFU_5_NC: now also IC1.E10 (RFU_5); no longer IC1.E10 (RFU_5)
- net RFU_6_NC: now also IC1.F10 (RFU_6); no longer IC1.F10 (RFU_6)
- net RFU_7_NC: now also IC1.G3 (RFU_7); no longer IC1.G3 (RFU_7)
- net RFU_8_NC: now also IC1.G10 (RFU_8); no longer IC1.G10 (RFU_8)
- net RFU_9_NC: now also IC1.K6 (RFU_9); no longer IC1.K6 (RFU_9)
- net nRST: now also IC1.K5 (RST_N); no longer IC1.K5 (RST_N)
- net at C22.2: now also IC1.C2 (VDDI); no longer IC1.C2 (VDDI)
- net VDD renamed +3V3
- net +3V3: now also IC1.C6 (VCCQ_1), IC1.E6 (VCC_1), IC1.F5 (VCC_2), IC1.J10 (VCC_3), IC1.K9 (VCC_4), IC1.M4 (VCCQ_2), IC1.N4 (VCCQ_3), IC1.P3 (VCCQ_4), IC1.P5 (VCCQ_5); no longer IC1.C6 (VCCQ_1), IC1.E6 (VCC_1), IC1.F5 (VCC_2), IC1.J10 (VCC_3), IC1.K9 (VCC_4), IC1.M4 (VCCQ_2), IC1.N4 (VCCQ_3), IC1.P3 (VCCQ_4), IC1.P5 (VCCQ_5)
Other:
- note added: "Can tie VCCQ to 1.8 for slightly reduced power consumption Important note is to ensure that the STM32 IOs are also set at 1p8V"
Changed lines of the file:
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@@
 	(generator_version "10.0")
 	(paper "A4")
+	(text "Can tie VCCQ to 1.8 for slightly reduced power consumption\nImportant note is to ensure that the STM32 IOs are also set at 1p8V"
+		(exclude_from_sim no)
+		(at 157.734 18.542 0)
+		(effects
+			(font
+				(size 1.27 1.27)
+			)
+		)
+	)
 	(junction
 		(at 121.92 49.53)
@@
 	)
 	(symbol
+		(lib_id "power:+3V3")
+		(at 21.59 52.07 0)
+		(unit 1)
+		(body_style 1)
+		(exclude_from_sim no)
+		(in_bom yes)
+		(on_board yes)
+		(in_pos_files yes)
+		(dnp no)
+		(fields_autoplaced yes)
+		(property "Reference" "#PWR02"
+			(at 21.59 55.88 0)
+			(hide yes)
+			(show_name no)
+			(do_not_autoplace no)
+			(effects
+				(font
+					(size 1.27 1.27)
+				)
+			)
+		)
+		(property "Value" "+3V3"
+			(at 21.59 46.99 0)
+			(show_name no)
+			(do_not_autoplace no)
+			(effects
+				(font
+					(size 1.27 1.27)
+				)
+			)
+		)
+		(property "Footprint" ""
+			(at 21.59 52.07 0)
+			(hide yes)
+			(show_name no)
+			(do_not_autoplace no)
+			(effects
+				(font
+					(size 1.27 1.27)
+				)
+			)
+		)
+		(property "Datasheet" ""
+			(at 21.59 52.07 0)
+			(hide yes)
+			(show_name no)
+			(do_not_autoplace no)
+			(effects
+				(font
+					(size 1.27 1.27)
+				)
+			)
+		)
+		(property "Description" "Power symbol creates a global label with name \"+3V3\""
+			(at 21.59 52.07 0)
+			(hide yes)
+			(show_name no)
+			(do_not_autoplace no)
+			(effects
+				(font
+					(size 1.27 1.27)
+				)
+			)
+		)
+		(pin "1"
+		)
+		(instances
+			(project "hardware"
+				(path "/a19f636f-b28d-4c43-b96a-b02383edd3eb/66e2f96f-c2f9-49fe-949d-95863aff4e55/b52766f3-1fa1-442f-884d-496f9ef14a5d"
+					(reference "#PWR02")
+					(unit 1)
+				)
+			)
+		)
+	)
+	(symbol
 		(lib_id "Device:C")
 		(at 67.31 62.23 0)
@@
 	)
 	(symbol
-		(lib_id "power:VDD")
+		(lib_id "power:+3V3")
 		(at 21.59 24.13 0)
 		(unit 1)
@@
 		(dnp no)
 		(fields_autoplaced yes)
-		(property "Reference" "#PWR042"
+		(property "Reference" "#PWR01"
 			(at 21.59 27.94 0)
 			(hide yes)
@@
 			)
 		)
-		(property "Value" "VDD"
+		(property "Value" "+3V3"
 			(at 21.59 19.05 0)
 			(show_name no)
@@
 			)
 		)
-		(property "Description" "Power symbol creates a global label with name \"VDD\""
+		(property "Description" "Power symbol creates a global label with name \"+3V3\""
 			(at 21.59 24.13 0)
 			(hide yes)
@@
 			(project "hardware"
 				(path "/a19f636f-b28d-4c43-b96a-b02383edd3eb/66e2f96f-c2f9-49fe-949d-95863aff4e55/b52766f3-1fa1-442f-884d-496f9ef14a5d"
-					(reference "#PWR042")
+					(reference "#PWR01")
 					(unit 1)
 				)
@@
 	)
 	(symbol
-		(lib_id "power:VDD")
-		(at 121.92 29.21 0)
-		(unit 1)
-		(body_style 1)
-		(exclude_from_sim no)
-		(in_bom yes)
-		(on_board yes)
-		(in_pos_files yes)
-		(dnp no)
-		(fields_autoplaced yes)
-		(property "Reference" "#PWR044"
-			(at 121.92 33.02 0)
-			(hide yes)
-			(show_name no)
-			(do_not_autoplace no)
-			(effects
-				(font
-					(size 1.27 1.27)
-				)
-			)
-		)
-		(property "Value" "VDD"
-			(at 121.92 24.13 0)
-			(show_name no)
-			(do_not_autoplace no)
-			(effects
-				(font
-					(size 1.27 1.27)
-				)
-			)
-		)
-		(property "Footprint" ""
-			(at 121.92 29.21 0)
-			(hide yes)
-			(show_name no)
-			(do_not_autoplace no)
-			(effects
-				(font
-					(size 1.27 1.27)
-				)
-			)
-		)
-		(property "Datasheet" ""
-			(at 121.92 29.21 0)
-			(hide yes)
-			(show_name no)
-			(do_not_autoplace no)
-			(effects
-				(font
-					(size 1.27 1.27)
-				)
-			)
-		)
-		(property "Description" "Power symbol creates a global label with name \"VDD\""
-			(at 121.92 29.21 0)
-			(hide yes)
-			(show_name no)
-			(do_not_autoplace no)
-			(effects
-				(font
-					(size 1.27 1.27)
-				)
-			)
-		)
-		(pin "1"
-		)
-		(instances
-			(project "hardware"
-				(path "/a19f636f-b28d-4c43-b96a-b02383edd3eb/66e2f96f-c2f9-49fe-949d-95863aff4e55/b52766f3-1fa1-442f-884d-496f9ef14a5d"
-					(reference "#PWR044")
-					(unit 1)
-				)
-			)
-		)
-	)
-	(symbol
 		(lib_id "power:GND")
 		(at 40.64 68.58 0)
@@
 	)
 	(symbol
-		(lib_id "power:VDD")
-		(at 21.59 52.07 0)
+		(lib_id "power:GND")
+		(at 41.91 43.18 0)
 		(unit 1)
 		(body_style 1)
@@
 		(dnp no)
 		(fields_autoplaced yes)
-		(property "Reference" "#PWR043"
-			(at 21.59 55.88 0)
+		(property "Reference" "#PWR032"
+			(at 41.91 49.53 0)
 			(hide yes)
 			(show_name no)
@@
 			)
 		)
-		(property "Value" "VDD"
-			(at 21.59 46.99 0)
+		(property "Value" "GND"
+			(at 41.91 48.26 0)
 			(show_name no)
 			(do_not_autoplace no)
@@
 		)
 		(property "Footprint" ""
-			(at 21.59 52.07 0)
+			(at 41.91 43.18 0)
 			(hide yes)
 			(show_name no)
@@
 		)
 		(property "Datasheet" ""
-			(at 21.59 52.07 0)
+			(at 41.91 43.18 0)
 			(hide yes)
 			(show_name no)
@@
 			)
 		)
-		(property "Description" "Power symbol creates a global label with name \"VDD\""
-			(at 21.59 52.07 0)
+		(property "Description" "Power symbol creates a global label with name \"GND\" , ground"
+			(at 41.91 43.18 0)
 			(hide yes)
 			(show_name no)
@@
 			(project "hardware"
 				(path "/a19f636f-b28d-4c43-b96a-b02383edd3eb/66e2f96f-c2f9-49fe-949d-95863aff4e55/b52766f3-1fa1-442f-884d-496f9ef14a5d"
-					(reference "#PWR043")
+					(reference "#PWR032")
 					(unit 1)
 				)
@@
 	)
 	(symbol
-		(lib_id "power:GND")
-		(at 41.91 43.18 0)
+		(lib_id "Device:C")
+		(at 27.94 62.23 0)
 		(unit 1)
 		(body_style 1)
@@
 		(dnp no)
 		(fields_autoplaced yes)
-		(property "Reference" "#PWR032"
-			(at 41.91 49.53 0)
-			(hide yes)
+		(property "Reference" "C25"
+			(at 31.75 60.9599 0)
 			(show_name no)
 			(do_not_autoplace no)
@@
 					(size 1.27 1.27)
 				)
+				(justify left)
 			)
 		)
-		(property "Value" "GND"
-			(at 41.91 48.26 0)
+		(property "Value" "100nF"
+			(at 31.75 63.4999 0)
 			(show_name no)
 			(do_not_autoplace no)
@@
 					(size 1.27 1.27)
 				)
+				(justify left)
 			)
 		)
 		(property "Footprint" ""
-			(at 41.91 43.18 0)
+			(at 28.9052 66.04 0)
 			(hide yes)
 			(show_name no)
@@
 		)
 		(property "Datasheet" ""
-			(at 41.91 43.18 0)
+			(at 27.94 62.23 0)
 			(hide yes)
 			(show_name no)
@@
 			)
 		)
-		(property "Description" "Power symbol creates a global label with name \"GND\" , ground"
-			(at 41.91 43.18 0)
+		(property "Description" "Unpolarized capacitor"
+			(at 27.94 62.23 0)
 			(hide yes)
 			(show_name no)
@@
 		(pin "1"
 		)
+		(pin "2"
+		)
 		(instances
 			(project "hardware"
 				(path "/a19f636f-b28d-4c43-b96a-b02383edd3eb/66e2f96f-c2f9-49fe-949d-95863aff4e55/b52766f3-1fa1-442f-884d-496f9ef14a5d"
-					(reference "#PWR032")
+					(reference "C25")
 					(unit 1)
 				)
@@
 	)
 	(symbol
-		(lib_id "Device:C")
-		(at 27.94 62.23 0)
+		(lib_id "power:+3V3")
+		(at 121.92 29.21 0)
 		(unit 1)
 		(body_style 1)
@@
 		(dnp no)
 		(fields_autoplaced yes)
-		(property "Reference" "C25"
-			(at 31.75 60.9599 0)
+		(property "Reference" "#PWR03"
+			(at 121.92 33.02 0)
+			(hide yes)
 			(show_name no)
 			(do_not_autoplace no)
@@
 					(size 1.27 1.27)
 				)
-				(justify left)
 			)
 		)
-		(property "Value" "100nF"
-			(at 31.75 63.4999 0)
+		(property "Value" "+3V3"
+			(at 121.92 24.13 0)
 			(show_name no)
 			(do_not_autoplace no)
@@
 					(size 1.27 1.27)
 				)
-				(justify left)
 			)
 		)
 		(property "Footprint" ""
-			(at 28.9052 66.04 0)
+			(at 121.92 29.21 0)
 			(hide yes)
 			(show_name no)
@@
 		)
 		(property "Datasheet" ""
-			(at 27.94 62.23 0)
+			(at 121.92 29.21 0)
 			(hide yes)
 			(show_name no)
@@
 			)
 		)
-		(property "Description" "Unpolarized capacitor"
-			(at 27.94 62.23 0)
+		(property "Description" "Power symbol creates a global label with name \"+3V3\""
+			(at 121.92 29.21 0)
 			(hide yes)
 			(show_name no)
@@
 		(pin "1"
 		)
-		(pin "2"
-		)
 		(instances
 			(project "hardware"
 				(path "/a19f636f-b28d-4c43-b96a-b02383edd3eb/66e2f96f-c2f9-49fe-949d-95863aff4e55/b52766f3-1fa1-442f-884d-496f9ef14a5d"
-					(reference "C25")
+					(reference "#PWR03")
 					(unit 1)
 				)

Commit message: Changing barometer, STM32 and power rails
Other:
- note added: "TODO: VCC must be 3p3, VCCQ can be 1p8"
Changed lines of the file:
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@@
 	(generator_version "10.0")
 	(paper "A4")
+	(text "TODO:\nVCC must be 3p3, VCCQ can be 1p8"
+		(exclude_from_sim no)
+		(at 178.562 169.672 0)
+		(effects
+			(font
+				(size 1.27 1.27)
+			)
+			(justify left)
+		)
+	)
 	(text "Can tie VCCQ to 1.8 for slightly reduced power consumption\nImportant note is to ensure that the STM32 IOs are also set at 1p8V"
 		(exclude_from_sim no)

Commit message: Added optical front end submodule and reconnected to STM32
Connections:
- net +3V3: no longer C25.1, C26.1, C27.1, C28.1, C29.1, IC1.C6 (VCCQ_1), IC1.M4 (VCCQ_2), IC1.N4 (VCCQ_3), IC1.P3 (VCCQ_4), IC1.P5 (VCCQ_5)
- new net +1V8: C25.1, C26.1, C27.1, C28.1, C29.1, IC1.C6 (VCCQ_1), IC1.M4 (VCCQ_2), IC1.N4 (VCCQ_3), IC1.P3 (VCCQ_4), IC1.P5 (VCCQ_5)

Commit message: Contemplating switching back to the 64LQFP
Other:
- note added: "What's going on with VDDI?"
Changed lines of the file:
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@@
+		)
+	)
+	(text "What's going on with VDDI?"
+		(exclude_from_sim no)
+		(at 87.884 23.368 0)
+		(effects
+			(font
+				(size 1.27 1.27)
+			)
+			(justify left)
 		)
 	)
