File: hardware/Bluetooth_Module.kicad_sch (KiCad schematic)
At the start: 7 parts, among them IC4 453-00171R, Y2 ECS-.327-6-12R-TR

Commit message: Changing barometer, STM32 and power rails
Other:
- note added: "TODO: 3p3 compatible only"
Changed lines of the file:
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@@
 	(generator_version "10.0")
 	(paper "A4")
+	(text "TODO:\n3p3 compatible only"
+		(exclude_from_sim no)
+		(at 178.308 170.18 0)
+		(effects
+			(font
+				(size 1.27 1.27)
+			)
+			(justify left)
+		)
+	)
 	(text "Open drain output on the STM32"
 		(exclude_from_sim no)

Commit message: Added level translator, connected all misc GPIO. Ensured that 64QLFP has support for 1.8V
Parts:
- C33, C34: value C -> 0.1uF
Connections:
- net +3V3: no longer C34.1, IC4.2 (VDDIO)
- new net +1V8: C34.1, IC4.2 (VDDIO)
Other:
- moved on the sheet: C33, C34
