File: hardware/STM32_64LQFP.kicad_sch (KiCad schematic)
At the start: 32 parts, among them J1 Conn_ARM_SWD_TagConnect_TC203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, U1 STM32U595RJTxQ, Y1 ECS-.327-6-12R-TR

Commit message: Added level translator, connected all misc GPIO. Ensured that 64QLFP has support for 1.8V
Connections:
- net PA2 is gone; now on net LPUART1_TX: U1.16 (PA2)
- net PA5 is gone; now on net SPI1_SCK: U1.21 (PA5)
- net PB10 is gone; now on net LPUART1_RX: U1.27 (PB10)
- net PB13 is gone; now on net LPUART1_CTS: U1.34 (PB13)
- net PC2 is gone; now on net SPI3_CS1: U1.10 (PC2)
- net LPUART1_CTS: no longer U1.22 (PA6)
- net LPUART1_RX: no longer U1.17 (PA3)
- net LPUART1_TX: no longer U1.9 (PC1)
- net SPI1_CS1: no longer U1.45 (PA12)
- net SPI1_MISO: no longer U1.44 (PA11)
- net SPI1_SCK: no longer U1.15 (PA1)
- net SPI3_CS1: no longer U1.40 (PC9)
- net SPI3_CS2: now also U1.15 (PA1); no longer U1.38 (PC7)
- net +3V3 renamed +1V8
- net PA0 renamed SDMMC2_CMD
- net PB14 renamed SDMMC2_D0
- net SDMMC1_CK renamed PC12
- net SDMMC1_CMD renamed PD2
- net SDMMC1_D0 renamed PC8
- new net PA11: U1.44 (PA11)
- new net PA12: U1.45 (PA12)
- new net PA3: U1.17 (PA3)
- new net PA6: U1.22 (PA6)
- new net PC7: U1.38 (PC7)
- new net PC9: U1.40 (PC9)
- new net SDMMC2_CK: U1.9 (PC1)
